File: CloudControlPCB/Schematic.brd (EAGLE design)
At the start: 57.1 x 61.9 mm, 31 parts, among them J1 AUDIO_JACK_TRRSSMD_RA, U1 LPC4088FBD208, U2 SGTL5000XNLA3R2, U3 LD1117S33CTR, X1 PHB_1MM27_2X05_SNT

Commit message: fixed JTAG on PCB
Parts:
- removed J5: (no value), SparkFun-Connectors:1X02
- moved R5 46.4 mm to (52.3, 80.8), turned to 180 degrees
- moved R2 2.48 mm to (33.0, 37.9)
- moved R1 2.28 mm to (29.0, 38.0)
Connections:
- removed net N$21: J5.2, U2.8
- removed net N$22: J5.1, U2.9
- net 3.3V: now also R5.2; no longer R5.1
- net N$16: now also R5.1, U1.110; no longer R5.2, U1.8, X1.10
- net N$18: now also X1.10
Routing:
- net N$18: track 10.7 -> 48.7 mm
- net N$16: track 37.8 -> 3.85 mm, vias 1 -> 0
- net N$22: track 17.7 -> 0.00 mm, vias 1 -> 0
- net N$21: track 15.3 -> 0.00 mm, vias 1 -> 0
- net N$13: track 29.8 -> 30.7 mm
- net 3.3V: track 47.3 -> 48.2 mm, vias 16 -> 15
Other:
- board text removed: "LineL"
- board text removed: "LineR"
